Commit message: sensors working correctly

File: src/autobot_description/urdf/autobot.urdf.xacro (robot description, xacro)
@@ -31,5 +31,5 @@
     <parent link="base_footprint" />
     <child link="base_link" />
-    <origin xyz="0 0 0.03" rpy="0 0 0" />
+    <!-- <origin xyz="0 0 0.03" rpy="0 0 0" /> -->
   </joint>
   <!-- Link laser_frame -->
@@ -59,5 +59,5 @@
   <!-- Joint from base_link to laser_frame -->
   <joint name="laser_frame_joint" type="fixed">
-    <origin xyz="-0 -0 0.2355" rpy="3.14159 -0 0" />
+    <origin xyz="-0 -0 0.2380" rpy="0 -0 0" />
     <parent link="base_link" />
     <child link="laser_frame" />
@@ -203,5 +203,5 @@
     <!-- Part rgbd_camera_link -->
     <visual>
-      <origin xyz="0 0.17 0.288" rpy="1.5708 1.5708 0" />
+      <origin xyz="-0.288 0 -0.17" rpy="0 0 0" />
       <geometry>
         <mesh filename="package://autobot_description/meshes/robot/rgbd_camera_link.stl" />
@@ -212,5 +212,5 @@
     </visual>
     <collision>
-      <origin xyz="0 0.17 0.288" rpy="1.5708 1.5708 0" />
+      <origin xyz="-0.288 0 -0.17" rpy="0 0 0" />
       <geometry>
         <mesh filename="package://autobot_description/meshes/robot/rgbd_camera_link.stl" />
@@ -220,8 +220,8 @@
   <!-- Joint from base_link to rgbd_camera_link -->
   <joint name="rgbd_camera_joint" type="fixed">
-    <origin xyz="0.288 0 0.17" rpy="-1.5708 -0 1.5708" />
+    <origin xyz="0.288 0 0.17" rpy="0 0 0" />
     <parent link="base_link" />
     <child link="rgbd_camera_link" />
-    <axis xyz="0 0 1" />
+    <axis xyz="0 0 -1" />
     <limit effort="10" velocity="10" />
   </joint>
@@ -230,4 +230,5 @@
     <sensor name="lidar_sensor" type="gpu_lidar">
       <topic>scan</topic>
+      <frame_id>laser_frame</frame_id>
       <update_rate>10</update_rate>
       <always_on>true</always_on>
@@ -249,8 +250,13 @@
         </scan>
         <range>
-          <min>0.20</min>
-          <max>30.0</max>
-          <resolution>0.013</resolution>
+          <min>0.05</min>
+          <max>20</max>
+          <resolution>0.01</resolution>
         </range>
+        <noise>
+          <type>gaussian</type>
+          <mean>0.0</mean>
+          <stddev>0.001</stddev>
+        </noise>
       </ray>
       <gz_frame_id>laser_frame</gz_frame_id>
@@ -261,12 +267,12 @@
     <sensor name="rgbd_camera" type="rgbd_camera">
       <camera>
-        <horizontal_fov>1.5184</horizontal_fov>
+        <horizontal_fov>2.094</horizontal_fov>
         <image>
-          <width>424</width>
-          <height>240</height>
+          <width>1080</width>
+          <height>720</height>
         </image>
         <clip>
-          <near>0.05</near>
-          <far>1.5</far>
+          <near>0.01</near>
+          <far>8</far>
         </clip>
       </camera>
@@ -274,5 +280,5 @@
       <gz_frame_id>rgbd_camera_depth_optical_frame</gz_frame_id>
       <topic>rgbd_camera</topic>
-      <update_rate>2</update_rate>
+      <update_rate>10</update_rate>
       <visualize>true</visualize>
     </sensor>

Commit message: lidar working, going to do the mapping

File: src/autobot_description/urdf/autobot.urdf.xacro (robot description, xacro)
@@ -6,7 +6,7 @@
     <inertial>
       <origin xyz="-0.000645097 1.49348e-05 0.123911" rpy="0 0 0" />
-      <mass value="19.3771" />
-      <inertia ixx="0.656608" ixy="-1.63412e-05" ixz="2.74753e-05" iyy="0.740294" iyz="2.27431e-05"
-        izz="1.21202" />
+      <mass value="58.1313" />
+      <inertia ixx="1.969824" ixy="-4.90236e-05" ixz="8.24259e-05" iyy="2.220882" iyz="6.82293e-05"
+        izz="3.63606" />
     </inertial>
     <!-- Part base_link -->
@@ -284,4 +284,13 @@
     </sensor>
   </gazebo>
+  <!-- IMU Sensor setup -->
+  <xacro:include
+    filename="$(find autobot_description)/urdf/sensors/imu.urdf.xacro" />
+  <xacro:imu_sensor
+    parent="base_link"
+    frame_id="imu"
+    xyz_offset="0 0 0"
+    rpy_offset="0 0 0"
+    topic_name="imu/data" />
   <xacro:include
     filename="$(find autobot_description)/urdf/control/velocity_control_plugin.urdf.xacro" />

Commit message: robot docking done, now moving closer to final

File: src/autobot_description/urdf/autobot.urdf.xacro (robot description, xacro)
@@ -6,7 +6,6 @@
     <inertial>
       <origin xyz="-0.000645097 1.49348e-05 0.123911" rpy="0 0 0" />
-      <mass value="58.1313" />
-      <inertia ixx="1.969824" ixy="-4.90236e-05" ixz="8.24259e-05" iyy="2.220882" iyz="6.82293e-05"
-        izz="3.63606" />
+      <mass value="19.3771"/>
+      <inertia ixx="0.656608" ixy="-1.63412e-05" ixz="2.74753e-05" iyy="0.740294" iyz="2.27431e-05" izz="1.21202"/>
     </inertial>
     <!-- Part base_link -->
@@ -211,10 +210,10 @@
       </material>
     </visual>
-    <collision>
+    <!-- <collision>
       <origin xyz="-0.288 0 -0.17" rpy="0 0 0" />
       <geometry>
         <mesh filename="package://autobot_description/meshes/robot/rgbd_camera_link.stl" />
       </geometry>
-    </collision>
+    </collision> -->
   </link>
   <!-- Joint from base_link to rgbd_camera_link -->
@@ -225,4 +224,11 @@
     <axis xyz="0 0 -1" />
     <limit effort="10" velocity="10" />
+  </joint>
+  <!-- Optical frame for the camera to match standard computer vision orientation -->
+  <link name="rgbd_camera_depth_optical_frame" />
+  <joint name="rgbd_camera_depth_optical_joint" type="fixed">
+    <origin xyz="0.05 0 0" rpy="-1.57079632679 0 -1.57079632679" />
+    <parent link="rgbd_camera_link" />
+    <child link="rgbd_camera_depth_optical_frame" />
   </joint>
   <!-- Laser gazebo setup -->
@@ -266,13 +272,14 @@
   <gazebo reference="rgbd_camera_link">
     <sensor name="rgbd_camera" type="rgbd_camera">
+      <pose>0.05 0 0 0 0 0</pose>
       <camera>
-        <horizontal_fov>2.094</horizontal_fov>
+        <horizontal_fov>2.1</horizontal_fov>
         <image>
-          <width>1080</width>
-          <height>720</height>
+          <width>424</width>
+          <height>240</height>
         </image>
         <clip>
-          <near>0.01</near>
-          <far>8</far>
+          <near>0.05</near>
+          <far>5</far>
         </clip>
       </camera>
@@ -280,5 +287,5 @@
       <gz_frame_id>rgbd_camera_depth_optical_frame</gz_frame_id>
       <topic>rgbd_camera</topic>
-      <update_rate>10</update_rate>
+      <update_rate>5</update_rate>
       <visualize>true</visualize>
     </sensor>
